Commit message: AI optimized working snapshot

File: delta_robot_description/models/model.urdf (robot description, URDF)
Before this commit: robot delta_robot, 28 links, 27 joints
Joints:
- joint jbf1: limit lower=-2.00713 upper=2.00713 effort=2 velocity=25 -> lower=-2.00713 upper=2.00713 effort=2 velocity=11.1
- joint jbf2: limit lower=-2.00713 upper=2.00713 effort=2 velocity=25 -> lower=-2.00713 upper=2.00713 effort=2 velocity=11.1
- joint jbf3: limit lower=-2.00713 upper=2.00713 effort=2 velocity=25 -> lower=-2.00713 upper=2.00713 effort=2 velocity=11.1
