Commit message: feat: enhance delta robot GUI and simulation
- Updated delta_robot_gui.launch.py to include new launch arguments for move_to_pose_service, play_demo_trajectory_service, motion_demo_service, and qt_qpa_platform.
- Modified delta_robot.rviz configuration to improve visualization settings and added new markers for trajectory visualization.
- Introduced plotter3d.py for 3D trajectory plotting with enhanced QoS settings and dynamic parameter handling.
- Added MoveToPose service definition to deltarobot_interfaces for improved motion control.
- Expanded DeltaJointVels and DeltaJoints message definitions to include additional joint velocities and positions.

File: delta_robot_description/models/model_high.sdf.xacro (robot description, xacro)
@@ -396,4 +396,5 @@
         <!-- World anchor -->
         <link name="world_link">
+            <pose>0 0 0 0 0 ${pi/2}</pose>
             <self_collide>false</self_collide>
             <inertial>
@@ -413,5 +414,5 @@
             <self_collide>false</self_collide>
             <static>true</static>
-            <pose>0 0 -0.059454 0 0 0</pose>
+            <pose>0 0 -0.059454 0 0 ${pi/2}</pose>
             <inertial>
                 <pose>0 0 0 0 0 0</pose>
@@ -610,5 +611,5 @@
         <link name="bevel_gear_ee">
             <self_collide>false</self_collide>
-            <pose>0 -0.00006 -0.14741 ${pi/2} 0 0.0829</pose>
+            <pose>0 0 -0.14741 ${pi/2} 0 0.0829</pose>
             <inertial>
                 <mass>0.0619505392</mass>
@@ -627,4 +628,8 @@
                 <xacro:material_black_pla/>
             </visual>
+        </link>
+        <link name="end_effector_pin">
+            <self_collide>false</self_collide>
+            <pose relative_to="bevel_gear_ee">0 -0.012 0 ${pi/2} -0.0829 0   </pose>
         </link>
         <!-- Virtual pivot constraints ─-->
@@ -717,9 +722,10 @@
         </plugin>
         <!-- Differential mechanism joints -->
-        <xacro:fixed_joint    name="end_effector_to_differential_c_arm"  parent="end_effector"       child="differential_c_arm"/>
+        <xacro:fixed_joint    name="end_effector_to_differential_c_arm"   parent="end_effector"       child="differential_c_arm"/>
         <xacro:revolute_joint name="differential_T_joint"                 parent="differential_c_arm" child="differentialT"  ax="1" ay=" 0" az="0"/>
-        <xacro:revolute_joint name="differential_pinion_joint_1"          parent="differential_c_arm" child="bevel_pinion_1" ax="0" ay=" 1" az="0"/>
-        <xacro:revolute_joint name="differential_pinion_joint_2"          parent="differential_c_arm" child="bevel_pinion_2" ax="0" ay=" 1" az="0"/>
+        <xacro:revolute_joint name="differential_pinion_joint_2"          parent="differential_c_arm" child="bevel_pinion_1" ax="0" ay=" 1" az="0"/>
+        <xacro:revolute_joint name="differential_pinion_joint_1"          parent="differential_c_arm" child="bevel_pinion_2" ax="0" ay=" 1" az="0"/>
         <xacro:revolute_joint name="differential_EE_joint"                parent="differentialT"      child="bevel_gear_ee"  ax="0" ay="-1" az="0"/>
+        <xacro:fixed_joint    name="end_effector_pin_joint"                     parent="bevel_gear_ee"      child="end_effector_pin"/>
         <!-- ROS 2 CONTROL -->
         <ros2_control name="GazeboSimSystem" type="system">

Commit message: Updated Model and removed sensor integration

File: delta_robot_description/models/model_high.sdf.xacro (robot description, xacro)
@@ -1,13 +1,16 @@
 <?xml version='1.0' encoding='utf-8'?>
 <sdf xmlns:xacro="http://www.ros.org/wiki/xacro" version="1.7">
-    <!-- PROPERTIES-->
-    <!-- Mesh package base-path. -->
+    <!-- ══════════════════════════════════════════════════════════
+         PROPERTIES
+    ══════════════════════════════════════════════════════════ -->
     <xacro:property name="meshes" value="package://delta_robot_description/meshes"/>
-    <!-- MATERIAL MACROS -->
+    <!-- ══════════════════════════════════════════════════════════
+         MATERIAL MACROS
+    ══════════════════════════════════════════════════════════ -->
     <xacro:macro name="material_aluminium">
         <material>
             <ambient>0.2  0.2  0.2  1</ambient>
             <diffuse>0.3  0.3  0.3  1</diffuse>
-            <specular>0.95 0.95 0.95 1</specular>
+            <specular>1.0  1.0  1.0  1</specular>
         </material>
     </xacro:macro>
@@ -33,11 +36,4 @@
         </material>
     </xacro:macro>
-    <xacro:macro name="material_grey_pla">
-        <material>
-            <ambient>0.15 0.15 0.15 1</ambient>
-            <diffuse>0.4  0.4  0.4  1</diffuse>
-            <specular>0.05 0.05 0.05 1</specular>
-        </material>
-    </xacro:macro>
     <xacro:macro name="material_black_pla">
         <material>
@@ -47,4 +43,11 @@
         </material>
     </xacro:macro>
+    <xacro:macro name="material_orange_pla">
+        <material>
+            <ambient>0.4  0.15 0.0  1</ambient>
+            <diffuse>1.0  0.4  0.0  1</diffuse>
+            <specular>0.1  0.1  0.1  1</specular>
+        </material>
+    </xacro:macro>
     <xacro:macro name="material_black_abs">
         <material>
@@ -61,5 +64,9 @@
         </material>
     </xacro:macro>
-    <!-- INERTIA MACROS -->
+    <!-- ══════════════════════════════════════════════════════════
+         INERTIA MACROS
+         Cross-terms (ixy/ixz/iyz) with |value| < 1e-9 are zeroed.
+         Negligible CoM pose offsets below the same threshold are also zeroed.
+    ══════════════════════════════════════════════════════════ -->
     <!-- Servo mount (×3) -->
     <xacro:macro name="inertial_servo_mount">
@@ -92,5 +99,5 @@
         </inertial>
     </xacro:macro>
-    <!-- Servo horn / free-horn (×6) -->
+    <!-- Servo horn / free-horn (×6) — driven (motor_joint_1/2/3 children) -->
     <xacro:macro name="inertial_servo_horn">
         <inertial>
@@ -122,5 +129,5 @@
         </inertial>
     </xacro:macro>
-    <!-- Upper pivot arm — pivot_arm_1 / 2 / 3 -->
+    <!-- Upper pivot arm (×3) -->
     <xacro:macro name="inertial_pivot_arm_upper">
         <inertial>
@@ -137,5 +144,5 @@
         </inertial>
     </xacro:macro>
-    <!-- Upper rod-cap — rod_cap_1 … rod_cap_6 -->
+    <!-- Upper rod-cap (×6) -->
     <xacro:macro name="inertial_rod_cap_upper">
         <inertial>
@@ -167,5 +174,5 @@
         </inertial>
     </xacro:macro>
-    <!-- Lower rod-cap — rod_cap_7 … rod_cap_12 -->
+    <!-- Lower rod-cap (×6) -->
     <xacro:macro name="inertial_rod_cap_lower">
         <inertial>
@@ -182,5 +189,5 @@
         </inertial>
     </xacro:macro>
-    <!-- Lower pivot arm — pivot_arm_4 / 5 / 6 -->
+    <!-- Lower pivot arm (×3) -->
     <xacro:macro name="inertial_pivot_arm_lower">
         <inertial>
@@ -197,20 +204,22 @@
         </inertial>
     </xacro:macro>
-    <!-- Bevel pinion (×2) -->
-    <xacro:macro name="inertial_bevel_pinion">
+    <!-- STS circular horn / bevel pinion (×2) — driven (differential_pinion_joint_1/2 children) -->
+    <xacro:macro name="inertial_sts_circular_horn">
         <inertial>
-            <mass>0.0190930454</mass>
-            <pose>-2.927e-07 0.00660778 2.94e-07 0 0 0</pose>
+            <mass>0.0039017949</mass>
+            <pose>0.0012497970 0 0 0 0 0</pose>
             <inertia>
-                <ixx>6.426e-07</ixx>
+                <ixx>1.4960e-07</ixx>
                 <ixy>0</ixy>
                 <ixz>0</ixz>
-                <iyy>7.99e-07</iyy>
+                <iyy>7.8203e-08</iyy>
                 <iyz>0</iyz>
-                <izz>6.426e-07</izz>
+                <izz>7.8203e-08</izz>
             </inertia>
         </inertial>
     </xacro:macro>
-    <!-- UTILITY MACROS -->
+    <!-- ══════════════════════════════════════════════════════════
+         UTILITY MACROS
+    ══════════════════════════════════════════════════════════ -->
     <!-- mesh_geometry -->
     <xacro:macro name="mesh_geometry" params="file">
@@ -222,5 +231,5 @@
         </geometry>
     </xacro:macro>
-    <!-- fixed_joint — type="fixed" with no pose element.    -->
+    <!-- fixed_joint -->
     <xacro:macro name="fixed_joint" params="name parent child">
         <joint name="${name}" type="fixed">
@@ -229,5 +238,5 @@
         </joint>
     </xacro:macro>
-    <!-- revolute_joint — type="revolute" -->
+    <!-- revolute_joint -->
     <xacro:macro name="revolute_joint" params="name parent child ax ay az">
         <joint name="${name}" type="revolute">
@@ -239,10 +248,12 @@
         </joint>
     </xacro:macro>
-    <!-- LINK MACROS -->
-    <!-- servo_mount_link -->
+    <!-- ══════════════════════════════════════════════════════════
+         LINK MACROS
+    ══════════════════════════════════════════════════════════ -->
+    <!-- servo_mount_link (×3) -->
     <xacro:macro name="servo_mount_link" params="n px py pz roll pitch yaw">
         <link name="servo_mount_${n}">
             <self_collide>false</self_collide>
-            <pose relative_to="delta_base-v1">${px} ${py} ${pz} ${roll} ${pitch} ${yaw}</pose>
+            <pose relative_to="delta_base">${px} ${py} ${pz} ${roll} ${pitch} ${yaw}</pose>
             <xacro:inertial_servo_mount/>
             <visual name="servo_mount_${n}_visual">
@@ -252,11 +263,11 @@
         </link>
     </xacro:macro>
-    <!-- servo_link -->
+    <!-- servo_link (×3) -->
     <xacro:macro name="servo_link" params="n">
         <link name="servo_${n}">
             <self_collide>false</self_collide>
-            <pose relative_to="servo_mount_${n}">0 0.0 -0.0213 ${pi/2} ${pi/2} 0</pose>
+            <pose relative_to="servo_mount_${n}">0 0 -0.0213 ${pi/2} ${pi/2} 0</pose>
             <xacro:inertial_servo/>
-            <visual name="servo_${n}">
+            <visual name="servo_${n}_visual">
                 <xacro:mesh_geometry file="servo.stl"/>
                 <xacro:material_black_abs/>
@@ -264,5 +275,5 @@
         </link>
     </xacro:macro>
-    <!-- servo_horn_link -->
+    <!-- servo_horn_link (×3) -->
     <xacro:macro name="servo_horn_link" params="n">
         <link name="servo_${n}_horn">
@@ -277,5 +288,5 @@
         </link>
     </xacro:macro>
-    <!-- servo_free_horn_link -->
+    <!-- servo_free_horn_link (×3) -->
     <xacro:macro name="servo_free_horn_link" params="n">
         <link name="servo_${n}_free_horn">
@@ -290,11 +301,11 @@
         </link>
     </xacro:macro>
-    <!-- bicep_link -->
+    <!-- bicep_link (×3) -->
     <xacro:macro name="bicep_link" params="n">
-        <link name="bicep${n}">
+        <link name="bicep_${n}">
             <self_collide>false</self_collide>
             <pose relative_to="servo_${n}_horn">0 0 0 0 0 ${-pi/2}</pose>
             <xacro:inertial_bicep/>
-            <visual name="bicep${n}_visual">
+            <visual name="bicep_${n}_visual">
                 <xacro:mesh_geometry file="bicep.stl"/>
                 <xacro:material_white_pla/>
@@ -302,5 +313,5 @@
         </link>
     </xacro:macro>
-    <!-- pivot_arm_upper_link -->
+    <!-- pivot_arm_upper_link (×3) -->
     <xacro:macro name="pivot_arm_upper_link" params="n px py pz roll pitch yaw">
         <link name="pivot_arm_${n}">
@@ -310,9 +321,9 @@
             <visual name="pivot_arm_${n}_visual">
                 <xacro:mesh_geometry file="pivot_arm.stl"/>
-                <xacro:material_grey_pla/>
-            </visual>
-        </link>
-    </xacro:macro>
-    <!-- rod_cap_upper_link -->
+                <xacro:material_white_pla/>
+            </visual>
+        </link>
+    </xacro:macro>
+    <!-- rod_cap_upper_link (×6) -->
     <xacro:macro name="rod_cap_upper_link" params="n relative_to z_offset">
         <link name="rod_cap_${n}">
@@ -327,9 +338,9 @@
         </link>
     </xacro:macro>
-    <!-- forearm_link -->
+    <!-- forearm_link (×6) -->
     <xacro:macro name="forearm_link" params="n relative_to">
         <link name="forearm_${n}">
             <self_collide>false</self_collide>
-            <pose relative_to="${relative_to}">0 0.195 0 ${pi/2} ${pi} 0</pose>
+            <pose relative_to="${relative_to}">0 0.258 0 ${pi/2} ${pi} 0</pose>
             <xacro:inertial_forearm/>
             <visual name="forearm_${n}_visual">
@@ -339,5 +350,5 @@
         </link>
     </xacro:macro>
-    <!-- rod_cap_lower_link -->
+    <!-- rod_cap_lower_link (×6) -->
     <xacro:macro name="rod_cap_lower_link" params="n relative_to roll">
         <link name="rod_cap_${n}">
@@ -351,5 +362,5 @@
         </link>
     </xacro:macro>
-    <!-- pivot_arm_lower_link -->
+    <!-- pivot_arm_lower_link (×3) -->
     <xacro:macro name="pivot_arm_lower_link" params="n relative_to">
         <link name="pivot_arm_${n}">
@@ -360,9 +371,97 @@
                 <pose>0 0 -0.016 0 0 0</pose>
                 <xacro:mesh_geometry file="pivot_arm.stl"/>
-                <xacro:material_grey_pla/>
-            </visual>
-        </link>
-    </xacro:macro>
-    <!-- virtual_pivot_link -->
+                <xacro:material_white_pla/>
+            </visual>
+        </link>
+    </xacro:macro>
+    <!-- detach_aux_link (×3) — massless aux links for DetachableJoint -->
+    <xacro:macro name="detach_aux_link" params="n">
+        <link name="rod_cap_${n}_aux">
+            <self_collide>false</self_collide>
+            <pose relative_to="rod_cap_${n}">0.0093 -0.005 0 0 0 0</pose>
+        </link>
+    </xacro:macro>
+    <!-- end_effector_side_plate_link (×2) -->
+    <xacro:macro name="end_effector_side_plate_link" params="n relative_to">
+        <link name="end_effector_side_plate_${n}">
+            <self_collide>false</self_collide>
+            <pose relative_to="${relative_to}">${((-1)**n) * 0.0346} 0.025 0 0 ${(n-2) * pi} 0</pose>
+            <inertial>
+                <mass>0.0225974194</mass>
+                <pose>-0.00016121771 -0.00081452055 0 0 0 0</pose>
+                <inertia>
+                    <ixx>1.0070887078e-05</ixx>
+                    <ixy>-1.8768434113e-08</ixy>
+                    <ixz>0</ixz>
+                    <iyy>3.3684942311e-06</iyy>
+                    <iyz>0</iyz>
+                    <izz>7.0797253681e-06</izz>
+                </inertia>
+            </inertial>
+            <visual name="end_effector_side_plate_${n}_visual">
+                <xacro:mesh_geometry file="end_effector_side_plate.stl"/>
+                <xacro:material_orange_pla/>
+            </visual>
+        </link>
+    </xacro:macro>
+    <!-- differential_servo_link (×2) — driven (differential_pinion_joint_1/2 parents) -->
+    <xacro:macro name="differential_servo" params="n relative_to">
+        <link name="differential_servo_${n}">
+            <self_collide>false</self_collide>
+            <pose relative_to="${relative_to}">0.0024 0.005 0 ${pi/2} ${pi/2} 0</pose>
+            <inertial>
+                <mass>0.0620599988</mass>
+                <pose>0 0.0079594816 0.0055633688 0 0 0</pose>
+                <inertia>
+                    <ixx>6.9884428428e-06</ixx>
+                    <ixy>0</ixy>
+                    <ixz>0</ixz>
+                    <iyy>3.6553944820e-06</iyy>
+                    <iyz>-3.4792797513e-08</iyz>
+                    <izz>4.7934769497e-06</izz>
+                </inertia>
+            </inertial>
+            <visual name="differential_servo_${n}_visual">
+                <xacro:mesh_geometry file="Feetech-STS2032.stl"/>
+                <xacro:material_black_abs/>
+            </visual>
+        </link>
+    </xacro:macro>
+    <!-- sts_circular_horn_link (×2) — driven (differential_pinion_joint_1/2 children) -->
+    <xacro:macro name="sts_circular_horn_link" params="n relative_to">
+        <link name="sts_circular_horn_${n}">
+            <self_collide>false</self_collide>
+            <pose relative_to="${relative_to}">0 -0.0110 0 0 0 ${pi/2}</pose>
+            <xacro:inertial_sts_circular_horn/>
+            <visual name="sts_circular_horn_${n}_visual">
+                <xacro:mesh_geometry file="sts_circular_horn.stl"/>
+                <xacro:material_black_pla/>
+            </visual>
+        </link>
+    </xacro:macro>
+    <!-- end_effector_pinion_link (×2) — driven -->
+    <xacro:macro name="end_effector_pinion" params="n relative_to">
+        <link name="end_effector_pinion_${n}">
+            <self_collide>false</self_collide>
+            <pose relative_to="${relative_to}">0.002 0 0 0 0 ${pi/2}</pose>
+            <inertial>
+                <mass>0.0031576875</mass>
+                <pose>0 0.0080716975 0 0 0 0</pose>
+                <inertia>
+                    <ixx>1.2058613504e-07</ixx>
+                    <ixy>0</ixy>
+                    <ixz>0</ixz>
+                    <iyy>1.2922906781e-07</iyy>
+                    <iyz>0</iyz>
+                    <izz>1.2058567290e-07</izz>
+                </inertia>
+            </inertial>
+            <visual name="end_effector_pinion_${n}_visual">
+                <xacro:mesh_geometry file="end_effector_pinion.stl"/>
+                <xacro:material_black_abs/>
+            </visual>
+        </link>
+    </xacro:macro>
+    <!-- virtual_pivot_link (×3) -->
     <xacro:macro name="virtual_pivot_link" params="n relative_to">
         <link name="virtual_pivot_${n}">
@@ -371,5 +470,8 @@
         </link>
     </xacro:macro>
-    <!-- motor_joint_set -->
+    <!-- ══════════════════════════════════════════════════════════
+         JOINT MACROS
+    ══════════════════════════════════════════════════════════ -->
+    <!-- motor_joint_set — driven revolute + mimic free-horn (×3) -->
     <xacro:macro name="motor_joint_set" params="n">
         <joint name="motor_joint_${n}" type="revolute">
@@ -392,5 +494,7 @@
         </joint>
     </xacro:macro>
-    <!-- MODEL -->
+    <!-- ══════════════════════════════════════════════════════════
+         MODEL
+    ══════════════════════════════════════════════════════════ -->
     <model name="delta_robot">
         <!-- World anchor -->
@@ -414,5 +518,5 @@
             <self_collide>false</self_collide>
             <static>true</static>
-            <pose>0 0 -0.059454 0 0 ${pi/2}</pose>
+            <pose relative_to="world_link">0 0 -0.059454 0 0 0</pose>
             <inertial>
                 <pose>0 0 0 0 0 0</pose>
@@ -427,8 +531,8 @@
                 </inertia>
             </inertial>
-            <collision name="Frame_collision">
+            <collision name="frame_collision">
                 <xacro:mesh_geometry file="frame.stl"/>
             </collision>
-            <visual name="Frame_visual">
+            <visual name="frame_visual">
                 <xacro:mesh_geometry file="frame.stl"/>
                 <xacro:material_black_aluminium/>
@@ -436,5 +540,5 @@
         </link>
         <!-- Delta base plate -->
-        <link name="delta_base-v1">
+        <link name="delta_base">
             <self_collide>false</self_collide>
             <pose>0 0 -0.01 0 0 0</pose>
@@ -451,44 +555,44 @@
                 </inertia>
             </inertial>
-            <visual name="delta_base-v1_visual">
+            <visual name="delta_base_visual">
                 <xacro:mesh_geometry file="delta_base-v1.stl"/>
                 <xacro:material_aluminium/>
             </visual>
         </link>
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
Commit message: refactor: restructure codebase by modularizing nodes into specific packages and cleaning up obsolete assets and scripts.

File: delta_robot_description/models/model_high.sdf.xacro (robot description, xacro)
@@ -481,4 +481,5 @@
                 <xyz>0 1 0</xyz>
             </axis>
+            <limit effort="2.0" velocity="11.1" lower="-3.14159" upper="3.14159"/>
         </joint>
         <joint name="motor_joint_${n}_free" type="revolute">
